Commit message: ouster description urdf changes

File: urdf/OS1-128.urdf.xacro (robot description, xacro)
@@ -55,5 +55,5 @@
       </visual>
     </link>
-    <link name="${imu_link}" />
+    <!-- <link name="${imu_link}" />
     <link name="${lidar_link}" />
     <joint name="${name}_imu_link_joint" type="fixed">
@@ -68,5 +68,5 @@
       <child link="${lidar_link}" />
       <origin xyz="0.0 0.0 0.03618" rpy="0 0 0" />
-    </joint>
+    </joint> -->
     <!-- Gazebo requires the ouster_gazebo_plugins package -->
     <gazebo reference="${name}">

Commit message: Adjusted Tf from os_sensor to os_lidar in urdf

File: urdf/OS1-128.urdf.xacro (robot description, xacro)
@@ -55,5 +55,5 @@
       </visual>
     </link>
-    <!-- <link name="${imu_link}" />
+    <link name="${imu_link}" />
     <link name="${lidar_link}" />
     <joint name="${name}_imu_link_joint" type="fixed">
@@ -67,6 +67,6 @@
       <parent link="${name}" />
       <child link="${lidar_link}" />
-      <origin xyz="0.0 0.0 0.03618" rpy="0 0 0" />
-    </joint> -->
+      <origin xyz="0.0 0.0 0.03618" rpy="0 0 3.142" />
+    </joint>
     <!-- Gazebo requires the ouster_gazebo_plugins package -->
     <gazebo reference="${name}">
